File: Commodore/C64/251469/userport.sch (KiCad schematic (older format))
At the start: 2 parts, among them CN2 User Port

Commit message: WIP
Connections:
- net labels added: ~PC2
- net labels removed: PC2
Changed lines of the file:
@@
 SP2
 Text HLabel 950  1800 0    50   Input ~ 0
-PC2
+~PC2
 Text HLabel 3000 1200 2    50   Output ~ 0
 ~FLAG2

Commit message: WIP
Parts:
- removed RP3: 3k3, symbol C64B:R_Network07_Split
Connections:
- wire segments 51 -> 38
Other:
- moved on the sheet: CN2
