File: Commodore/C64/251469/reset.sch (KiCad schematic (older format))
At the start: 11 parts, among them Q3 2SC1815, U20 LM556, U8 7406

Commit message: WIP
Parts:
- C39: value .1 μF -> 0.1 μF
Changed lines of the file:
@@
 EESchema Schematic File Version 4
 LIBS:C64B-cache
-EELAYER 29 0
+EELAYER 30 0
 EELAYER END
 $Descr A4 11693 8268
 encoding utf-8
-Sheet 3 15
+Sheet 14 15
 Title "Commodore 64 - Reset Section (schematic #251469)"
 Date "2019-07-16"
@@
 AR Path="/5D9CCECB/5D9D12F3" Ref="C39"  Part="1"
 F 0 "C39" V 1750 900 50  0000 L CNN
-F 1 ".1 μF" V 1950 850 50  0000 L CNN
+F 1 "0.1 μF" V 1950 850 50  0000 L CNN
 F 2 "" H 1850 950 50  0001 C CNN
 F 3 "~" H 1850 950 50  0001 C CNN
