File: Apple/Apple II/IIgs/ROM3 Schematic/RAM-9.sch (KiCad schematic (older format))
At the start: 11 parts

Commit message: Fixed rescue
Fixed a mistake with the libraries. Also adding back the cache.
Parts:
- U? (x8): symbol IIgs-Schematic-rescue:HMS511000-Apple_IIgs_Symbols -> IIgs-Schematic:HMS511000
- U? (x2): symbol IIgs-Schematic-rescue:IIgs-ROM-Apple_IIgs_Symbols -> IIgs-Schematic:IIgs-ROM
Changed lines of the file:
@@
 EESchema Schematic File Version 4
 LIBS:IIgs Schematic-cache
-EELAYER 26 0
+EELAYER 29 0
 EELAYER END
 $Descr A3 16535 11693
@@
 $EndDescr
 $Comp
-L IIgs-Schematic-rescue:HMS511000-Apple_IIgs_Symbols U?
+L IIgs-Schematic:HMS511000 U?
 U 1 1 5BF22D2A
 P 3450 2200
@@
 $EndComp
 $Comp
-L IIgs-Schematic-rescue:HMS511000-Apple_IIgs_Symbols U?
+L IIgs-Schematic:HMS511000 U?
 U 1 1 5BF22D4E
 P 5650 2200
@@
 $EndComp
 $Comp
-L IIgs-Schematic-rescue:HMS511000-Apple_IIgs_Symbols U?
+L IIgs-Schematic:HMS511000 U?
 U 1 1 5BF22D61
 P 7800 2200
@@
 $EndComp
 $Comp
-L IIgs-Schematic-rescue:HMS511000-Apple_IIgs_Symbols U?
+L IIgs-Schematic:HMS511000 U?
 U 1 1 5BF22D78
 P 9900 2200
@@
 $EndComp
 $Comp
-L IIgs-Schematic-rescue:HMS511000-Apple_IIgs_Symbols U?
+L IIgs-Schematic:HMS511000 U?
 U 1 1 5BF22D8D
 P 9950 5500
@@
 $EndComp
 $Comp
-L IIgs-Schematic-rescue:HMS511000-Apple_IIgs_Symbols U?
+L IIgs-Schematic:HMS511000 U?
 U 1 1 5BF22DAC
 P 7950 5500
@@
 $EndComp
 $Comp
-L IIgs-Schematic-rescue:HMS511000-Apple_IIgs_Symbols U?
+L IIgs-Schematic:HMS511000 U?
 U 1 1 5BF22DCC
 P 5700 5500
@@
 $EndComp
 $Comp
-L IIgs-Schematic-rescue:HMS511000-Apple_IIgs_Symbols U?
+L IIgs-Schematic:HMS511000 U?
 U 1 1 5BF22DF0
 P 3500 5450
@@
 $EndComp
 $Comp
-L IIgs-Schematic-rescue:IIgs-ROM-Apple_IIgs_Symbols U?
+L IIgs-Schematic:IIgs-ROM U?
 U 1 1 5BF22ECB
 P 3500 8900
@@
 $EndComp
 $Comp
-L IIgs-Schematic-rescue:IIgs-ROM-Apple_IIgs_Symbols U?
+L IIgs-Schematic:IIgs-ROM U?
 U 1 1 5BF22EF8
 P 6550 8900

Commit message: More work on Sound
Other edits to other pages
Parts:
- gave numbers to parts that had none: 11
Changed lines of the file:
@@
 $EndDescr
 $Comp
-L IIgs-Schematic:HMS511000 U?
+L IIgs-Schematic:HMS511000 UE8
 U 1 1 5BF22D2A
 P 3450 2200
-F 0 "U?" H 3550 3150 50  0000 C CNN
+F 0 "UE8" H 3550 3150 50  0000 C CNN
 F 1 "HMS511000" H 3700 3050 50  0000 C CNN
 F 2 "" H 3200 2950 50  0001 C CNN
@@
 $EndComp
 $Comp
-L IIgs-Schematic:HMS511000 U?
+L IIgs-Schematic:HMS511000 UE9
 U 1 1 5BF22D4E
 P 5650 2200
-F 0 "U?" H 5800 3150 50  0000 C CNN
+F 0 "UE9" H 5800 3150 50  0000 C CNN
 F 1 "HMS511000" H 5950 3050 50  0000 C CNN
 F 2 "" H 5400 2950 50  0001 C CNN
@@
 $EndComp
 $Comp
-L IIgs-Schematic:HMS511000 U?
+L IIgs-Schematic:HMS511000 UE10
 U 1 1 5BF22D61
 P 7800 2200
-F 0 "U?" H 7900 3150 50  0000 C CNN
+F 0 "UE10" H 7900 3150 50  0000 C CNN
 F 1 "HMS511000" H 8050 3050 50  0000 C CNN
 F 2 "" H 7550 2950 50  0001 C CNN
@@
 $EndComp
 $Comp
-L IIgs-Schematic:HMS511000 U?
+L IIgs-Schematic:HMS511000 UE11
 U 1 1 5BF22D78
 P 9900 2200
-F 0 "U?" H 10000 3150 50  0000 C CNN
+F 0 "UE11" H 10000 3150 50  0000 C CNN
 F 1 "HMS511000" H 10150 3050 50  0000 C CNN
 F 2 "" H 9650 2950 50  0001 C CNN
@@
 $EndComp
 $Comp
-L IIgs-Schematic:HMS511000 U?
+L IIgs-Schematic:HMS511000 UF11
 U 1 1 5BF22D8D
 P 9950 5500
-F 0 "U?" H 10050 6450 50  0000 C CNN
+F 0 "UF11" H 10050 6450 50  0000 C CNN
 F 1 "HMS511000" H 10200 6350 50  0000 C CNN
 F 2 "" H 9700 6250 50  0001 C CNN
@@
 $EndComp
 $Comp
-L IIgs-Schematic:HMS511000 U?
+L IIgs-Schematic:HMS511000 UF10
 U 1 1 5BF22DAC
 P 7950 5500
-F 0 "U?" H 8050 6450 50  0000 C CNN
+F 0 "UF10" H 8050 6450 50  0000 C CNN
 F 1 "HMS511000" H 8200 6350 50  0000 C CNN
 F 2 "" H 7700 6250 50  0001 C CNN
@@
 $EndComp
 $Comp
-L IIgs-Schematic:HMS511000 U?
+L IIgs-Schematic:HMS511000 UF9
 U 1 1 5BF22DCC
 P 5700 5500
-F 0 "U?" H 5800 6450 50  0000 C CNN
+F 0 "UF9" H 5800 6450 50  0000 C CNN
 F 1 "HMS511000" H 5950 6350 50  0000 C CNN
 F 2 "" H 5450 6250 50  0001 C CNN
@@
 $EndComp
 $Comp
-L IIgs-Schematic:HMS511000 U?
+L IIgs-Schematic:HMS511000 UF8
 U 1 1 5BF22DF0
 P 3500 5450
-F 0 "U?" H 3600 6400 50  0000 C CNN
+F 0 "UF8" H 3600 6400 50  0000 C CNN
 F 1 "HMS511000" H 3750 6300 50  0000 C CNN
 F 2 "" H 3250 6200 50  0001 C CNN
@@
 $EndComp
 $Comp
-L IIgs-Schematic:IIgs-ROM U?
+L IIgs-Schematic:IIgs-ROM UJ9
 U 1 1 5BF22ECB
 P 3500 8900
-F 0 "U?" H 3600 10000 50  0000 C CNN
+F 0 "UJ9" H 3600 10000 50  0000 C CNN
 F 1 "IIgs-ROM" H 3700 9900 50  0000 C CNN
 F 2 "" H 3250 9750 50  0001 C CNN
@@
 $EndComp
 $Comp
-L IIgs-Schematic:IIgs-ROM U?
+L IIgs-Schematic:IIgs-ROM UJ11
 U 1 1 5BF22EF8
 P 6550 8900
-F 0 "U?" H 6650 9950 50  0000 C CNN
+F 0 "UJ11" H 6650 9950 50  0000 C CNN
 F 1 "IIgs-ROM" H 6750 9850 50  0000 C CNN
 F 2 "" H 6300 9750 50  0001 C CNN
@@
 $EndComp
 $Comp
-L 74xx:74LS74 U?
+L 74xx:74LS74 UJ6
 U 1 1 5BF22FB9
 P 4750 7300
-F 0 "U?" H 4850 7650 50  0000 C CNN
+F 0 "UJ6" H 4850 7650 50  0000 C CNN
 F 1 "74LS74" H 4900 7550 50  0000 C CNN
 F 2 "" H 4750 7300 50  0001 C CNN
