File: Apple/Apple II/IIgs/ROM3 Schematic/Slots-7.sch (KiCad schematic (older format))
At the start: 22 parts, among them J1 Apple_II_Slot, J2 Apple_II_Slot, J3 Apple_II_Slot, J4 Apple_II_Slot, J5 Apple_II_Slot, J6 Apple_II_Slot, J7 Apple_II_Slot

Commit message: Fixed rescue
Fixed a mistake with the libraries. Also adding back the cache.
Parts:
- J1, J2, J3, J4, J5, J6, J7: symbol IIgs-Schematic-rescue:Apple_II_Slot-Apple_IIgs_Symbols -> IIgs-Schematic:Apple_II_Slot
- UC10: symbol IIgs-Schematic-rescue:Slotmaker-Apple_IIgs_Symbols -> IIgs-Schematic:Slotmaker
- UD5: symbol IIgs-Schematic-rescue:HCT245-Apple_IIgs_Symbols -> IIgs-Schematic:HCT245
Changed lines of the file:
@@
 EESchema Schematic File Version 4
 LIBS:IIgs Schematic-cache
-EELAYER 26 0
+EELAYER 29 0
 EELAYER END
 $Descr A3 16535 11693
@@
 $EndDescr
 $Comp
-L IIgs-Schematic-rescue:Apple_II_Slot-Apple_IIgs_Symbols J1
+L IIgs-Schematic:Apple_II_Slot J1
 U 1 1 5BF21608
 P 6200 4300
@@
 $EndComp
 $Comp
-L IIgs-Schematic-rescue:Apple_II_Slot-Apple_IIgs_Symbols J2
+L IIgs-Schematic:Apple_II_Slot J2
 U 1 1 5BF21629
 P 8900 4300
@@
 $EndComp
 $Comp
-L IIgs-Schematic-rescue:Apple_II_Slot-Apple_IIgs_Symbols J3
+L IIgs-Schematic:Apple_II_Slot J3
 U 1 1 5BF21642
 P 11600 4300
@@
 $EndComp
 $Comp
-L IIgs-Schematic-rescue:Apple_II_Slot-Apple_IIgs_Symbols J4
+L IIgs-Schematic:Apple_II_Slot J4
 U 1 1 5BF2165E
 P 14300 4300
@@
 $EndComp
 $Comp
-L IIgs-Schematic-rescue:Apple_II_Slot-Apple_IIgs_Symbols J5
+L IIgs-Schematic:Apple_II_Slot J5
 U 1 1 5BF2167B
 P 6200 7550
@@
 $EndComp
 $Comp
-L IIgs-Schematic-rescue:Apple_II_Slot-Apple_IIgs_Symbols J6
+L IIgs-Schematic:Apple_II_Slot J6
 U 1 1 5BF2169A
 P 8900 7550
@@
 $EndComp
 $Comp
-L IIgs-Schematic-rescue:Apple_II_Slot-Apple_IIgs_Symbols J7
+L IIgs-Schematic:Apple_II_Slot J7
 U 1 1 5BF216B7
 P 11600 7550
@@
 $EndComp
 $Comp
-L IIgs-Schematic-rescue:Slotmaker-Apple_IIgs_Symbols UC10
+L IIgs-Schematic:Slotmaker UC10
 U 1 1 5BF217D2
 P 2600 4900
@@
 $EndComp
 $Comp
-L IIgs-Schematic-rescue:HCT245-Apple_IIgs_Symbols UD5
+L IIgs-Schematic:HCT245 UD5
 U 1 1 5BF2195F
 P 2650 8500

Commit message: Finish CYA Page
First draft of CYA page. Also switched all passives to use the _Small symbol variant.
Parts:
- R112, R113, R197: symbol Device:R -> Device:R_Small
Other:
- note added: "Verify if this is the XOR from the CYA Page"
Changed lines of the file:
@@
 	1850 8950 2250 8950
 $Comp
-L Device:R R113
+L Device:R_Small R113
 U 1 1 5E438F86
 P 4150 2350
@@
 $EndComp
 $Comp
-L Device:R R112
+L Device:R_Small R112
 U 1 1 5E43903C
 P 4150 2700
@@
 Text Label 4650 2350 2    50   ~ 0
 RDY.H
-Wire Wire Line
-	4300 2350 4650 2350
-Wire Wire Line
-	4300 2700 4650 2700
 Text Label 4650 2700 2    50   ~ 0
 NMI.L
 Wire Wire Line
-	4000 2700 3850 2700
-Wire Wire Line
 	3850 2700 3850 2350
-Wire Wire Line
-	3850 2350 4000 2350
 $Comp
 L power:+5V #PWR?
@@
 	1700 2450 2200 2450
 $Comp
-L Device:R R197
+L Device:R_Small R197
 U 1 1 5E979E74
 P 2450 2450
@@
 	0    1    1    0
 $EndComp
-Wire Wire Line
-	2300 2450 2200 2450
 Connection ~ 2200 2450
 Text Label 2950 2450 2    50   ~ 0
 M2BADD
 Wire Wire Line
-	2600 2450 2950 2450
+	4250 2350 4650 2350
+Wire Wire Line
+	4250 2700 4650 2700
+Wire Wire Line
+	3850 2350 4050 2350
+Wire Wire Line
+	3850 2700 4050 2700
+Wire Wire Line
+	2200 2450 2350 2450
+Wire Wire Line
+	2550 2450 2950 2450
+Text Notes 750  1950 0    50   ~ 0
+Verify if this is the XOR from the CYA Page
 $EndSCHEMATC

Commit message: Finished Sound Page (and the rest!)
Cleaned up Capacitor page with polarized caps.
Stil need to make some global labels (optional)
Thank you chat! -> 2020-07-19
Other:
- note added: "Global labels not shown"
Changed lines of the file:
@@
 Text Notes 750  1950 0    50   ~ 0
 Verify if this is the XOR from the CYA Page
+Text Notes 2300 700  0    50   ~ 0
+Global labels not shown
 $EndSCHEMATC
