File: Tandy-RS/TRS-80 Color Computer/Color Computer 2/26-313x/sam.sch (KiCad schematic (older format))
At the start: 26 parts, among them IC10 74LS02, IC11 74LS138, IC22 MC6883, IC5 74LS273, IC6 74LS244, X1 14.31818 MHz

Commit message: Finish drawing initial version of Coco2 schematic
Connections:
- net labels added: D[0..7], MD[0..7], Z0, Z1, Z2, Z3, Z4, Z5, Z6, Z7, Z[0..7]
- net labels removed: D
- wire segments 176 -> 179
- no-connect marks 1 -> 3
Changed lines of the file:
@@
 encoding utf-8
 Sheet 6 8
-Title ""
-Date ""
-Rev ""
-Comp ""
-Comment1 ""
+Title "TRS-80 Color Computer 2 (26-3134 / 26-3136) - SAM"
+Date "2020-10-14"
+Rev "0.1"
+Comp "Tandy Corporation"
+Comment1 "Based on \"Service Manual TRS-80 Color Computer 2 NTSC Version\" pp. 87"
 Comment2 ""
 Comment3 ""
-Comment4 ""
+Comment4 "Kicad schematic capture by troysbucket"
 $EndDescr
 $Comp
@@
 	1750 1400 3300 1400
 $Comp
-L power:GND #PWR?
+L power:GND #PWR0142
 U 1 1 5F7FA689
 P 4150 4950
-F 0 "#PWR?" H 4150 4700 50  0001 C CNN
+F 0 "#PWR0142" H 4150 4700 50  0001 C CNN
 F 1 "GND" H 4150 4800 50  0000 C CNN
 F 2 "" H 4150 4950 50  0001 C CNN
@@
 $EndComp
 $Comp
-L power:GND #PWR?
+L power:GND #PWR0143
 U 1 1 5F7FAB39
 P 4950 1850
-F 0 "#PWR?" H 4950 1600 50  0001 C CNN
+F 0 "#PWR0143" H 4950 1600 50  0001 C CNN
 F 1 "GND" H 4950 1700 50  0000 C CNN
 F 2 "" H 4950 1850 50  0001 C CNN
 F 3 "" H 4950 1850 50  0001 C CNN
 	1    4950 1850
-	1    0    0    -1
-$EndComp
-$Comp
-L power:+5V #PWR?
-U 1 1 5F7FB028
-P 5650 1200
-F 0 "#PWR?" H 5650 1050 50  0001 C CNN
-F 1 "+5V" H 5650 1340 50  0000 C CNN
-F 2 "" H 5650 1200 50  0001 C CNN
-F 3 "" H 5650 1200 50  0001 C CNN
-	1    5650 1200
 	1    0    0    -1
 $EndComp
@@
 $EndComp
 $Comp
-L power:GND #PWR?
+L power:GND #PWR0145
 U 1 1 5F7FE837
 P 4650 1850
-F 0 "#PWR?" H 4650 1600 50  0001 C CNN
+F 0 "#PWR0145" H 4650 1600 50  0001 C CNN
 F 1 "GND" H 4650 1700 50  0000 C CNN
 F 2 "" H 4650 1850 50  0001 C CNN
@@
 $EndComp
 Wire Wire Line
-	4150 2050 4150 1400
-Wire Wire Line
-	4150 1400 4650 1400
+	4150 1400 4350 1400
 Wire Wire Line
 	5450 1400 5650 1400
@@
 $EndComp
 $Comp
-L power:GND #PWR?
+L power:GND #PWR0146
 U 1 1 5F8088CA
 P 3450 4450
-F 0 "#PWR?" H 3450 4200 50  0001 C CNN
+F 0 "#PWR0146" H 3450 4200 50  0001 C CNN
 F 1 "GND" H 3450 4300 50  0000 C CNN
 F 2 "" H 3450 4450 50  0001 C CNN
@@
 $EndComp
 $Comp
-L power:GND #PWR?
+L power:GND #PWR0147
 U 1 1 5F808C5D
 P 3000 4450
-F 0 "#PWR?" H 3000 4200 50  0001 C CNN
+F 0 "#PWR0147" H 3000 4200 50  0001 C CNN
 F 1 "GND" H 3000 4300 50  0000 C CNN
 F 2 "" H 3000 4450 50  0001 C CNN
@@
 $EndComp
 $Comp
-L power:GND #PWR?
+L power:GND #PWR0148
 U 1 1 5F808ECF
 P 2000 4450
-F 0 "#PWR?" H 2000 4200 50  0001 C CNN
+F 0 "#PWR0148" H 2000 4200 50  0001 C CNN
 F 1 "GND" H 2000 4300 50  0000 C CNN
 F 2 "" H 2000 4450 50  0001 C CNN
@@
 	4650 2250 4900 2250
 Text Label 4700 2250 0    50   ~ 0
-A0
+Z0
 Wire Wire Line
 	4900 2350 4650 2350
@@
 	4900 3050 4650 3050
 Text Label 4700 2350 0    50   ~ 0
-A1
+Z1
 Text Label 4700 2450 0    50   ~ 0
-A2
+Z2
 Text Label 4700 2550 0    50   ~ 0
-A3
+Z3
 Text Label 4700 2650 0    50   ~ 0
-A4
+Z4
 Text Label 4700 2750 0    50   ~ 0
-A5
+Z5
 Text Label 4700 2850 0    50   ~ 0
-A6
+Z6
 Text Label 4700 3050 0    50   ~ 0
-A7
+Z7
 Entry Wire Line
 	4900 2250 5000 2150
@@
 $EndComp
 $Comp
-L power:GND #PWR?
+L power:GND #PWR0149
 U 1 1 5F870D13
 P 5400 4050
-F 0 "#PWR?" H 5400 3800 50  0001 C CNN
+F 0 "#PWR0149" H 5400 3800 50  0001 C CNN
 F 1 "GND" H 5400 3900 50  0000 C CNN
 F 2 "" H 5400 4050 50  0001 C CNN
@@
 $EndComp
 $Comp
-L power:GND #PWR?
+L power:GND #PWR0150
 U 1 1 5F87100B
 P 5650 4050
-F 0 "#PWR?" H 5650 3800 50  0001 C CNN
+F 0 "#PWR0150" H 5650 3800 50  0001 C CNN
 F 1 "GND" H 5650 3900 50  0000 C CNN
 F 2 "" H 5650 4050 50  0001 C CNN
@@
 Connection ~ 5650 3550
 $Comp
-L power:+5V #PWR?
+L power:+5V #PWR0151
 U 1 1 5F8897E2
 P 2350 6000
-F 0 "#PWR?" H 2350 5850 50  0001 C CNN
+F 0 "#PWR0151" H 2350 5850 50  0001 C CNN
 F 1 "+5V" H 2350 6140 50  0000 C CNN
 F 2 "" H 2350 6000 50  0001 C CNN
@@
 $EndComp
 $Comp
-L power:GND #PWR?
+L power:GND #PWR0152
 U 1 1 5F889FF6
 P 2350 7150
-F 0 "#PWR?" H 2350 6900 50  0001 C CNN
+F 0 "#PWR0152" H 2350 6900 50  0001 C CNN
 F 1 "GND" H 2350 7000 50  0000 C CNN
 F 2 "" H 2350 7150 50  0001 C CNN
@@
 $EndComp
 $Comp
-L power:GND #PWR?
+L power:GND #PWR0153
 U 1 1 5F88A332
 P 1100 7150
-F 0 "#PWR?" H 1100 6900 50  0001 C CNN
+F 0 "#PWR0153" H 1100 6900 50  0001 C CNN
 F 1 "GND" H 1100 7000 50  0000 C CNN
 F 2 "" H 1100 7150 50  0001 C CNN
@@
 $EndComp
 $Comp
-L power:+5V #PWR?
+L power:+5V #PWR0164
 U 1 1 5F89A182
 P 6300 3900
-F 0 "#PWR?" H 6300 3750 50  0001 C CNN
+F 0 "#PWR0164" H 6300 3750 50  0001 C CNN
 F 1 "+5V" H 6300 4040 50  0000 C CNN
 F 2 "" H 6300 3900 50  0001 C CNN
@@
 $EndComp
 $Comp
-L power:GND #PWR?
+L power:GND #PWR0165
 U 1 1 5F89A929
 P 6850 4100
-F 0 "#PWR?" H 6850 3850 50  0001 C CNN
+F 0 "#PWR0165" H 6850 3850 50  0001 C CNN
 F 1 "GND" H 6850 3950 50  0000 C CNN
 F 2 "" H 6850 4100 50  0001 C CNN
@@
 $EndComp
 $Comp
-L power:GND #PWR?
+L power:GND #PWR0166
 U 1 1 5F89AB35
 P 6300 5450
-F 0 "#PWR?" H 6300 5200 50  0001 C CNN
+F 0 "#PWR0166" H 6300 5200 50  0001 C CNN
 F 1 "GND" H 6300 5300 50  0000 C CNN
 F 2 "" H 6300 5450 50  0001 C CNN
@@
 $EndComp
 $Comp
-L power:+5V #PWR?
+L power:+5V #PWR0167
 U 1 1 5F8B4531
 P 5150 4800
-F 0 "#PWR?" H 5150 4650 50  0001 C CNN
+F 0 "#PWR0167" H 5150 4650 50  0001 C CNN
 F 1 "+5V" H 5150 4940 50  0000 C CNN
 F 2 "" H 5150 4800 50  0001 C CNN
@@
 	4650 3350 6150 3350
 Text HLabel 1750 800  0    50   BiDi ~ 0
-D
+D[0..7]
 Wire Bus Line
 	1750 800  6000 800
@@
 $EndComp
 $Comp
-L power:+5V #PWR?
+L power:+5V #PWR0168
 U 1 1 5F9B7D15
 P 9250 1600
-F 0 "#PWR?" H 9250 1450 50  0001 C CNN
+F 0 "#PWR0168" H 9250 1450 50  0001 C CNN
 F 1 "+5V" H 9250 1740 50  0000 C CNN
 F 2 "" H 9250 1600 50  0001 C CNN
@@
 $EndComp
 $Comp
-L power:GND #PWR?
+L power:GND #PWR0169
 U 1 1 5F9B8273
 P 9850 1750
-F 0 "#PWR?" H 9850 1500 50  0001 C CNN
+F 0 "#PWR0169" H 9850 1500 50  0001 C CNN
 F 1 "GND" H 9850 1600 50  0000 C CNN
 F 2 "" H 9850 1750 50  0001 C CNN
@@
 $EndComp
 $Comp
-L power:GND #PWR?
+L power:GND #PWR0170
 U 1 1 5F9B85FF
 P 9250 3450
-F 0 "#PWR?" H 9250 3200 50  0001 C CNN
+F 0 "#PWR0170" H 9250 3200 50  0001 C CNN
 F 1 "GND" H 9250 3300 50  0000 C CNN
 F 2 "" H 9250 3450 50  0001 C CNN
@@
 $EndComp
 $Comp
-L power:GND #PWR?
+L power:GND #PWR0171
 U 1 1 5F78D75B
 P 9250 5850
-F 0 "#PWR?" H 9250 5600 50  0001 C CNN
+F 0 "#PWR0171" H 9250 5600 50  0001 C CNN
 F 1 "GND" H 9250 5700 50  0000 C CNN
 F 2 "" H 9250 5850 50  0001 C CNN
@@
 $EndComp
 $Comp
-L power:+5V #PWR?
+L power:+5V #PWR0172
 U 1 1 5F78D761
 P 9250 3950
-F 0 "#PWR?" H 9250 3800 50  0001 C CNN
+F 0 "#PWR0172" H 9250 3800 50  0001 C CNN
 F 1 "+5V" H 9250 4090 50  0000 C CNN
 F 2 "" H 9250 3950 50  0001 C CNN
@@
 $EndComp
 $Comp
-L power:GND #PWR?
+L power:GND #PWR0173
 U 1 1 5F78D767
 P 9650 4150
-F 0 "#PWR?" H 9650 3900 50  0001 C CNN
+F 0 "#PWR0173" H 9650 3900 50  0001 C CNN
 F 1 "GND" H 9650 4000 50  0000 C CNN
 F 2 "" H 9650 4150 50  0001 C CNN
@@
 $EndComp
 $Comp
-L power:+5V #PWR?
+L power:+5V #PWR0174
 U 1 1 5F78D76D
 P 8500 5700
-F 0 "#PWR?" H 8500 5550 50  0001 C CNN
+F 0 "#PWR0174" H 8500 5550 50  0001 C CNN
 F 1 "+5V" H 8500 5840 50  0000 C CNN
 F 2 "" H 8500 5700 50  0001 C CNN
@@
 	6800 4650 6900 4650
 $Comp
-L power:GND #PWR?
+L power:GND #PWR0175
 U 1 1 5F8C443D
 P 7300 5450
-F 0 "#PWR?" H 7300 5200 50  0001 C CNN
+F 0 "#PWR0175" H 7300 5200 50  0001 C CNN
 F 1 "GND" H 7300 5300 50  0000 C CNN
 F 2 "" H 7300 5450 50  0001 C CNN
@@
 	7550 4650 7300 4650
 Connection ~ 7300 4650
+Text Label 7700 1950 0    50   ~ 0
+MD[0..7]
+Text Label 5450 2100 0    50   ~ 0
+Z[0..7]
+NoConn ~ 1900 6350
+NoConn ~ 1900 6750
+Wire Wire Line
+	1900 6750 1800 6750
+Wire Wire Line
+	1900 6350 1800 6350
+$Comp
+L power:+5V #PWR0144
+U 1 1 5F905C7F
+P 5650 1200
+F 0 "#PWR0144" H 5650 1050 50  0001 C CNN
+F 1 "+5V" H 5650 1340 50  0000 C CNN
+F 2 "" H 5650 1200 50  0001 C CNN
+F 3 "" H 5650 1200 50  0001 C CNN
+	1    5650 1200
+	1    0    0    -1
+$EndComp
+Wire Wire Line
+	4150 1400 4150 2050
+$Comp
+L power:PWR_FLAG #FLG0102
+U 1 1 5F920A1F
+P 4350 1400
+F 0 "#FLG0102" H 4350 1475 50  0001 C CNN
+F 1 "PWR_FLAG" H 4350 1550 50  0000 C CNN
+F 2 "" H 4350 1400 50  0001 C CNN
+F 3 "~" H 4350 1400 50  0001 C CNN
+	1    4350 1400
+	1    0    0    -1
+$EndComp
+Connection ~ 4350 1400
+Wire Wire Line
+	4350 1400 4650 1400
 Wire Bus Line
 	5000 2100 5000 2950
