File: Apple/Apple IIGS/IIgs/ROM3 Schematic/Video-3.sch (KiCad schematic (older format))
At the start: 107 parts, among them J10 Video Connector, J11 RCA MONO OUT, Q1 2n3904, Q2 2n3904, Q3 2n3904, Y1 32.768 kHz

Commit message: Clean-up after detailed circuit analysis - Fixed Reference to library in project file - Fixed BABUS tags on HCT245 (had wrong nets) - Flipped HCT245 circuits on MEGAII page to better match In/Out flow - Changed HCT245 symbol to move enable and DIR to better match In/Out Flow - Changed HCT245 into multi-unit symbol to put VCC/GND pins on Unit B - Fixed MEGAII designator - Fixed ADBUS nets on HCT245 (should be ABUS!) - Added notes with lessons learned from circuit deep-dive
Parts:
- H1: symbol IIgs-Schematic:Video_Sync -> IIgs-Schematic-rescue:Video_Sync-IIgs-Schematic
- H2, H3, H4: symbol IIgs-Schematic:VideoThingy -> IIgs-Schematic-rescue:VideoThingy-IIgs-Schematic
- J11: symbol IIgs-Schematic:Conn_Coaxial_2_Shield_Pins -> IIgs-Schematic-rescue:Conn_Coaxial_2_Shield_Pins-IIgs-Schematic
- TF1: symbol IIgs-Schematic:CapacitiveTransformer -> IIgs-Schematic-rescue:CapacitiveTransformer-IIgs-Schematic
- UB2: symbol IIgs-Schematic:MC1377 -> IIgs-Schematic-rescue:MC1377-IIgs-Schematic
- UD4: symbol IIgs-Schematic:SERCLK -> IIgs-Schematic-rescue:SERCLK-IIgs-Schematic
- UF2: symbol IIgs-Schematic:VGC -> IIgs-Schematic-rescue:VGC-IIgs-Schematic
Other:
- note added: "All clocks derived from\n28.636360 MHz Xtal\n\nUnclear who generates 14M:\nMEGA-II or VGC\n\nPH0 and PH2 not entirely clear"
- note added: "H2, H3, and H4 form\nDAC for RGB video"
- note added: "MDBUSx goes back to MEGA-II"
- note added: "STRETCH:\nEvery 65 clocks, A2 must have 1\nlonger clock period. For each\nHorizontal line."
- note added: "VIDx - 12-bit binary values for RGB"
Changed lines of the file:
@@
 $EndDescr
 $Comp
-L IIgs-Schematic:VGC UF2
+L IIgs-Schematic-rescue:VGC-IIgs-Schematic UF2
 U 1 1 5BF1D843
 P 4100 4500
@@
 Connection ~ 10900 8750
 $Comp
-L IIgs-Schematic:MC1377 UB2
+L IIgs-Schematic-rescue:MC1377-IIgs-Schematic UB2
 U 1 1 5BF1DCA3
 P 11100 6900
@@
 	12100 7000 12150 7000
 $Comp
-L IIgs-Schematic:VideoThingy H2
+L IIgs-Schematic-rescue:VideoThingy-IIgs-Schematic H2
 U 1 1 5EE8F7E3
 P 6450 1900
@@
 $EndComp
 $Comp
-L IIgs-Schematic:VideoThingy H3
+L IIgs-Schematic-rescue:VideoThingy-IIgs-Schematic H3
 U 1 1 5EE8FCB7
 P 6450 2700
@@
 $EndComp
 $Comp
-L IIgs-Schematic:VideoThingy H4
+L IIgs-Schematic-rescue:VideoThingy-IIgs-Schematic H4
 U 1 1 5EE900C8
 P 6450 3450
@@
 $EndComp
 $Comp
-L IIgs-Schematic:Conn_Coaxial_2_Shield_Pins J11
+L IIgs-Schematic-rescue:Conn_Coaxial_2_Shield_Pins-IIgs-Schematic J11
 U 1 1 5F61A5F9
 P 15100 7150
@@
 J11-1
 $Comp
-L IIgs-Schematic:CapacitiveTransformer TF1
+L IIgs-Schematic-rescue:CapacitiveTransformer-IIgs-Schematic TF1
 U 1 1 5F6AFD3C
 P 14300 7100
@@
 $EndComp
 $Comp
-L IIgs-Schematic:SERCLK UD4
+L IIgs-Schematic-rescue:SERCLK-IIgs-Schematic UD4
 U 1 1 5F833608
 P 7500 9600
@@
 $EndComp
 $Comp
-L IIgs-Schematic:Video_Sync H1
+L IIgs-Schematic-rescue:Video_Sync-IIgs-Schematic H1
 U 1 1 5EF591B0
 P 10150 2400
@@
 Text Notes 3650 900  0    50   ~ 0
 Off-Page symbols not show on the UF2
+Text Notes 6050 1500 0    50   ~ 0
+H2, H3, and H4 form\nDAC for RGB video
+Text Notes 4700 3800 0    50   ~ 0
+VIDx - 12-bit binary values for RGB
+Text Notes 1650 4150 0    50   ~ 0
+MDBUSx goes back to MEGA-II
+Text Notes 650  5300 0    50   ~ 0
+All clocks derived from\n28.636360 MHz Xtal\n\nUnclear who generates 14M:\nMEGA-II or VGC\n\nPH0 and PH2 not entirely clear
+Text Notes 1350 4550 0    50   ~ 0
+STRETCH:\nEvery 65 clocks, A2 must have 1\nlonger clock period. For each\nHorizontal line.
 $EndSCHEMATC
