File: Apple/Apple IIGS/IIgs/ROM3 Schematic/CYA-Mem-1.kicad_sch (KiCad schematic)
At the start: 38 parts, among them J20 IIgs_Memory_Connector, U6 65SC816

Commit message: Formatting clean-up
Changed lines of the file:
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@@
   (title_block
     (title "CPU and Fast Memory Controller (CYA)")
+    (date "2023-01-28")
     (rev "2")
     (company "bald.ee/bitpreserve")
@@
     (stroke (width 0) (type default) (color 0 0 0 0))
   )
-  (bus_entry (at 386.715 196.85) (size 2.54 -2.54)
-    (stroke (width 0) (type default) (color 0 0 0 0))
-  )
-  (bus_entry (at 386.715 189.23) (size 2.54 -2.54)
-    (stroke (width 0) (type default) (color 0 0 0 0))
-  )
-  (bus_entry (at 386.715 186.69) (size 2.54 -2.54)
+  (bus_entry (at 358.775 176.53) (size 2.54 -2.54)
+    (stroke (width 0) (type default) (color 0 0 0 0))
+  )
+  (bus_entry (at 358.775 168.91) (size 2.54 -2.54)
+    (stroke (width 0) (type default) (color 0 0 0 0))
+  )
+  (bus_entry (at 358.775 166.37) (size 2.54 -2.54)
     (stroke (width 0) (type default) (color 0 0 0 0))
   )
@@
     (stroke (width 0) (type default) (color 0 0 0 0))
   )
-  (bus_entry (at 386.715 179.07) (size 2.54 -2.54)
-    (stroke (width 0) (type default) (color 0 0 0 0))
-  )
-  (bus_entry (at 386.715 184.15) (size 2.54 -2.54)
+  (bus_entry (at 358.775 158.75) (size 2.54 -2.54)
+    (stroke (width 0) (type default) (color 0 0 0 0))
+  )
+  (bus_entry (at 358.775 163.83) (size 2.54 -2.54)
     (stroke (width 0) (type default) (color 0 0 0 0))
   )
@@
     (stroke (width 0) (type default) (color 0 0 0 0))
   )
-  (bus_entry (at 386.715 199.39) (size 2.54 -2.54)
-    (stroke (width 0) (type default) (color 0 0 0 0))
-  )
-  (bus_entry (at 386.715 201.93) (size 2.54 -2.54)
+  (bus_entry (at 358.775 179.07) (size 2.54 -2.54)
+    (stroke (width 0) (type default) (color 0 0 0 0))
+  )
+  (bus_entry (at 358.775 181.61) (size 2.54 -2.54)
     (stroke (width 0) (type default) (color 0 0 0 0))
   )
@@
     (stroke (width 0) (type default) (color 0 0 0 0))
   )
-  (bus_entry (at 386.715 181.61) (size 2.54 -2.54)
+  (bus_entry (at 358.775 161.29) (size 2.54 -2.54)
     (stroke (width 0) (type default) (color 0 0 0 0))
   )
@@
     (stroke (width 0) (type default) (color 0 0 0 0))
   )
-  (bus_entry (at 386.715 194.31) (size 2.54 -2.54)
+  (bus_entry (at 358.775 173.99) (size 2.54 -2.54)
     (stroke (width 0) (type default) (color 0 0 0 0))
   )
@@
     (stroke (width 0) (type default) (color 0 0 0 0))
   )
-  (bus_entry (at 386.715 191.77) (size 2.54 -2.54)
+  (bus_entry (at 358.775 171.45) (size 2.54 -2.54)
     (stroke (width 0) (type default) (color 0 0 0 0))
   )
@@
     (stroke (width 0) (type default) (color 0 0 0 0))
   )
-  (wire (pts (xy 375.285 191.77) (xy 386.715 191.77))
+  (wire (pts (xy 347.345 171.45) (xy 358.775 171.45))
     (stroke (width 0) (type default) (color 0 0 0 0))
   )
@@
     (stroke (width 0) (type default) (color 0 0 0 0))
   )
-  (wire (pts (xy 386.715 179.07) (xy 375.285 179.07))
+  (wire (pts (xy 358.775 158.75) (xy 347.345 158.75))
     (stroke (width 0) (type default) (color 0 0 0 0))
   )
@@
     (stroke (width 0) (type default) (color 0 0 0 0))
   )
-  (wire (pts (xy 375.285 196.85) (xy 386.715 196.85))
+  (wire (pts (xy 347.345 176.53) (xy 358.775 176.53))
     (stroke (width 0) (type default) (color 0 0 0 0))
   )
@@
     (stroke (width 0) (type default) (color 0 0 0 0))
   )
-  (bus (pts (xy 389.255 176.53) (xy 389.255 179.07))
+  (bus (pts (xy 361.315 156.21) (xy 361.315 158.75))
     (stroke (width 0) (type default) (color 0 0 0 0))
   )
@@
     (stroke (width 0) (type default) (color 0 0 0 0))
   )
-  (bus (pts (xy 389.255 184.15) (xy 389.255 186.69))
+  (bus (pts (xy 361.315 163.83) (xy 361.315 166.37))
     (stroke (width 0) (type default) (color 0 0 0 0))
   )
@@
     (stroke (width 0) (type default) (color 0 0 0 0))
   )
-  (bus (pts (xy 389.255 194.31) (xy 389.255 196.85))
+  (bus (pts (xy 361.315 173.99) (xy 361.315 176.53))
     (stroke (width 0) (type default) (color 0 0 0 0))
   )
@@
     (stroke (width 0) (type default) (color 0 0 0 0))
   )
-  (bus (pts (xy 389.255 174.625) (xy 393.065 174.625))
+  (bus (pts (xy 361.315 154.305) (xy 365.125 154.305))
     (stroke (width 0) (type default) (color 0 0 0 0))
   )
@@
     (stroke (width 0) (type default) (color 0 0 0 0))
   )
-  (wire (pts (xy 386.715 189.23) (xy 375.285 189.23))
-    (stroke (width 0) (type default) (color 0 0 0 0))
-  )
-  (bus (pts (xy 389.255 196.85) (xy 389.255 199.39))
+  (wire (pts (xy 358.775 168.91) (xy 347.345 168.91))
+    (stroke (width 0) (type default) (color 0 0 0 0))
+  )
+  (bus (pts (xy 361.315 176.53) (xy 361.315 179.07))
     (stroke (width 0) (type default) (color 0 0 0 0))
   )
@@
     (stroke (width 0) (type default) (color 0 0 0 0))
   )
-  (wire (pts (xy 386.715 181.61) (xy 375.285 181.61))
-    (stroke (width 0) (type default) (color 0 0 0 0))
-  )
-  (wire (pts (xy 386.715 199.39) (xy 375.285 199.39))
+  (wire (pts (xy 358.775 161.29) (xy 347.345 161.29))
+    (stroke (width 0) (type default) (color 0 0 0 0))
+  )
+  (wire (pts (xy 358.775 179.07) (xy 347.345 179.07))
     (stroke (width 0) (type default) (color 0 0 0 0))
   )
@@
     (stroke (width 0) (type default) (color 0 0 0 0))
   )
-  (wire (pts (xy 375.285 186.69) (xy 386.715 186.69))
+  (wire (pts (xy 347.345 166.37) (xy 358.775 166.37))
     (stroke (width 0) (type default) (color 0 0 0 0))
   )
@@
     (stroke (width 0) (type default) (color 0 0 0 0))
   )
-  (bus (pts (xy 389.255 181.61) (xy 389.255 184.15))
-    (stroke (width 0) (type default) (color 0 0 0 0))
-  )
-  (bus (pts (xy 389.255 191.77) (xy 389.255 194.31))
+  (bus (pts (xy 361.315 161.29) (xy 361.315 163.83))
+    (stroke (width 0) (type default) (color 0 0 0 0))
+  )
+  (bus (pts (xy 361.315 171.45) (xy 361.315 173.99))
     (stroke (width 0) (type default) (color 0 0 0 0))
   )
@@
     (stroke (width 0) (type default) (color 0 0 0 0))
   )
-  (wire (pts (xy 375.285 184.15) (xy 386.715 184.15))
+  (wire (pts (xy 347.345 163.83) (xy 358.775 163.83))
     (stroke (width 0) (type default) (color 0 0 0 0))
   )
@@
     (stroke (width 0) (type default) (color 0 0 0 0))
   )
-  (bus (pts (xy 389.255 174.625) (xy 389.255 176.53))
+  (bus (pts (xy 361.315 154.305) (xy 361.315 156.21))
     (stroke (width 0) (type default) (color 0 0 0 0))
   )
@@
     (stroke (width 0) (type default) (color 0 0 0 0))
   )
-  (wire (pts (xy 386.715 194.31) (xy 375.285 194.31))
+  (wire (pts (xy 358.775 173.99) (xy 347.345 173.99))
     (stroke (width 0) (type default) (color 0 0 0 0))
   )
@@
     (stroke (width 0) (type default) (color 0 0 0 0))
   )
-  (wire (pts (xy 375.285 201.93) (xy 386.715 201.93))
+  (wire (pts (xy 347.345 181.61) (xy 358.775 181.61))
     (stroke (width 0) (type default) (color 0 0 0 0))
   )
@@
     (stroke (width 0) (type default) (color 0 0 0 0))
   )
-  (bus (pts (xy 389.255 186.69) (xy 389.255 189.23))
+  (bus (pts (xy 361.315 166.37) (xy 361.315 168.91))
     (stroke (width 0) (type default) (color 0 0 0 0))
   )
@@
     (stroke (width 0) (type default) (color 0 0 0 0))
   )
-  (bus (pts (xy 389.255 189.23) (xy 389.255 191.77))
+  (bus (pts (xy 361.315 168.91) (xy 361.315 171.45))
     (stroke (width 0) (type default) (color 0 0 0 0))
   )
@@
     (stroke (width 0) (type default) (color 0 0 0 0))
   )
-  (bus (pts (xy 389.255 179.07) (xy 389.255 181.61))
+  (bus (pts (xy 361.315 158.75) (xy 361.315 161.29))
     (stroke (width 0) (type default) (color 0 0 0 0))
   )
@@
     (effects (font (size 1.27 1.27)) (justify left bottom))
   )
-  (label "FRABUSD3" (at 375.285 186.69 0)
+  (label "FRABUSD3" (at 347.345 166.37 0)
     (effects (font (size 1.27 1.27)) (justify left bottom))
   )
@@
     (effects (font (size 1.27 1.27)) (justify left bottom))
   )
-  (label "FRABUSD2" (at 375.285 184.15 0)
-    (effects (font (size 1.27 1.27)) (justify left bottom))
-  )
-  (label "FRABUSD7" (at 375.285 196.85 0)
+  (label "FRABUSD2" (at 347.345 163.83 0)
+    (effects (font (size 1.27 1.27)) (justify left bottom))
+  )
+  (label "FRABUSD7" (at 347.345 176.53 0)
     (effects (font (size 1.27 1.27)) (justify left bottom))
   )
@@
     (effects (font (size 1.27 1.27)) (justify left bottom))
   )
-  (label "FRABUSD9" (at 375.285 201.93 0)
+  (label "FRABUSD9" (at 347.345 181.61 0)
     (effects (font (size 1.27 1.27)) (justify left bottom))
   )
@@
     (effects (font (size 1.27 1.27)) (justify left bottom))
   )
-  (label "FRABUSD8" (at 375.285 199.39 0)
+  (label "FRABUSD8" (at 347.345 179.07 0)
     (effects (font (size 1.27 1.27)) (justify left bottom))
   )
@@
     (effects (font (size 1.27 1.27)) (justify left bottom))
   )
-  (label "FRABUSD0" (at 375.285 179.07 0)
+  (label "FRABUSD0" (at 347.345 158.75 0)
     (effects (font (size 1.27 1.27)) (justify left bottom))
   )
@@
     (effects (font (size 1.27 1.27)) (justify left bottom))
   )
-  (label "FRABUSD5" (at 375.285 191.77 0)
+  (label "FRABUSD5" (at 347.345 171.45 0)
     (effects (font (size 1.27 1.27)) (justify left bottom))
   )
@@
     (effects (font (size 1.27 1.27)) (justify right bottom))
   )
-  (label "FRABUSD1" (at 375.285 181.61 0)
+  (label "FRABUSD1" (at 347.345 161.29 0)
     (effects (font (size 1.27 1.27)) (justify left bottom))
   )
@@
     (effects (font (size 1.27 1.27)) (justify left bottom))
   )
-  (label "FRABUSD6" (at 375.285 194.31 0)
+  (label "FRABUSD6" (at 347.345 173.99 0)
     (effects (font (size 1.27 1.27)) (justify left bottom))
   )
@@
     (effects (font (size 1.27 1.27)) (justify right bottom))
   )
-  (label "FRABUSD4" (at 375.285 189.23 0)
+  (label "FRABUSD4" (at 347.345 168.91 0)
     (effects (font (size 1.27 1.27)) (justify left bottom))
   )
@@
     (effects (font (size 1.27 1.27)) (justify right))
   )
-  (hierarchical_label "FRABUSD[9..0]" (shape output) (at 393.065 174.625 0)
+  (hierarchical_label "FRABUSD[9..0]" (shape output) (at 365.125 154.305 0)
     (effects (font (size 1.27 1.27)) (justify left))
   )
