File: Tandy-RS/TRS-80 Color Computer/Color Computer 2/26-313xA/coco2/coco2.sch (KiCad schematic (older format))
At the start: 7 parts, among them CN1 Conn_02x20_Odd_Even

Commit message: -updated pcb -updated some part numbers
Parts:
- C1: Manufacturer part# FG28C0G1H103JNT06 -> RDER71H104K0K1H03B; Vendor part# 445-173474-1-ND -> 490-8814-ND
Changed lines of the file:
@@
 F 1 ".1uF" H 1900 3900 50  0000 C CNN
 F 2 "Capacitor_THT:C_Disc_D4.7mm_W2.5mm_P5.00mm" H 2000 3800 50  0001 C CNN
-F 3 " https://product.tdk.com/info/en/catalog/datasheets/leadmlcc_halogenfree_fg_en.pdf?ref_disty=digikey" H 2000 3800 50  0001 C CNN
+F 3 " https://search.murata.co.jp/Ceramy/image/img/A01X/G101/ENG/RDE_X7R_250V-1kV_E.pdf" H 2000 3800 50  0001 C CNN
 F 4 "digikey" V 2000 3800 50  0001 C CNN "Vendor"
-F 5 "445-173474-1-ND" V 2000 3800 50  0001 C CNN "Vendor part#"
-F 6 "FG28C0G1H103JNT06" V 2000 3800 50  0001 C CNN "Manufacturer part#"
+F 5 "490-8814-ND" V 2000 3800 50  0001 C CNN "Vendor part#"
+F 6 "RDER71H104K0K1H03B" V 2000 3800 50  0001 C CNN "Manufacturer part#"
 	1    2000 3800
 	-1   0    0    1
