File: Apple/Apple IIe/Apple IIe (NTSC) - 050-0051-D/IO-2.kicad_sch (KiCad schematic)
At the start: 46 parts, among them J18 Conn_01x02, J19 Conn_01x02, J9 CASSETTE IN, Q5 MPSA13, X1 SolderJumper_2_Open, X2 SolderJumper_2_Bridged, X6 SolderJumper_2_Open

Commit message: Updated symbols, added power symbols for multi-units, and passed ERC!
Parts:
- C79: symbol Device:CP_Small -> Device:C_Polarized_Small
Changed lines of the file:
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@@
     )
   )
-  (symbol (lib_id "Device:CP_Small") (at 247.65 220.98 270) (unit 1)
+  (symbol (lib_id "Device:C_Polarized_Small") (at 247.65 220.98 270) (unit 1)
     (in_bom yes) (on_board yes) (dnp no)
     (property "Reference" "C79" (at 247.65 215.265 90)
@@
     )
     (property "Datasheet" "~" (at 260.35 226.06 90)
+      (effects (font (size 1.27 1.27)) hide)
+    )
+    (property "Sim.Device" "D" (at 260.35 226.06 0)
+      (effects (font (size 1.27 1.27)) hide)
+    )
+    (property "Sim.Pins" "1=K 2=A" (at 260.35 226.06 0)
       (effects (font (size 1.27 1.27)) hide)
     )
@@
       (effects (font (size 1.27 1.27)) hide)
     )
-    (property "Datasheet" "" (at 252.73 132.08 0)
-      (effects (font (size 1.27 1.27)) hide)
-    )
+    (property "Datasheet" "http://www.ti.com/lit/gpn/sn74ls02" (at 252.73 132.08 0)
+      (effects (font (size 1.27 1.27)) hide)
+    )

Commit message: Fixes #87
Connections:
- net ~{ENKBD}: now also UE12.18 (~{CE}); no longer UE12.16 (~{CE})
Changed lines of the file:
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@@
     (pin "15")
     (pin "16")
-    (pin "16")
+    (pin "18")
     (pin "19")
     (pin "2")
