File: Apple/Apple II+/AppleII+/Video Gen.kicad_sch (KiCad schematic)
At the start: 51 parts, among them J18 Aux Video, K14 VIDEO OUT, Q3 2N3904, Q6 2N3904

Commit message: Changed SOFT5-A2-8 and -11 to just SOFT5, based on Apple II Circuit Description Book
Parts:
- renumbered JP10 to JP14, JP11 to JP16
Connections:
- net SOFT5-A2-11 is gone; now on net SOFT5: A2.11
- net SOFT5-A2-8 is gone; now on net SOFT5: A2.8
Other:
- note added: ""The Apple II Circuit Description" shows multiple versions of this part of the schematic. V0 is much different than V1 and later. -baldee"
- note added: "From "The Apple II Circuit Description", page 152: Soft S-Rev.7 and earlier boards use high outputs of gates A2-8 and A2-11 instead of R28 to pull up unused logic inputs"
Changed lines of the file:
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@@
     (stroke (width 0) (type default))
   )
+  (wire (pts (xy 32.385 163.195) (xy 45.72 163.195))
+    (stroke (width 0) (type default))
+  )
   (wire (pts (xy 238.125 45.72) (xy 239.395 45.72))
     (stroke (width 0) (type default))
@@
     (stroke (width 0) (type default))
   )
-  (wire (pts (xy 387.35 51.435) (xy 370.84 51.435))
-    (stroke (width 0) (type default))
-  )
   (wire (pts (xy 373.38 116.205) (xy 377.19 116.205))
     (stroke (width 0) (type default))
@@
     (stroke (width 0) (type default))
   )
-  (wire (pts (xy 370.84 66.675) (xy 387.35 66.675))
-    (stroke (width 0) (type default))
-  )
   (wire (pts (xy 147.955 180.975) (xy 161.925 180.975))
     (stroke (width 0) (type default))
@@
     (stroke (width 0) (type default))
   )
+  (text "From \"The Apple II Circuit Description\", page 152:\nSoft S-Rev.7 and earlier boards use high outputs of gates A2-8 and A2-11\ninstead of R28 to pull up unused logic inputs"
+    (at 31.115 283.21 0)
+    (effects (font (size 1.27 1.27)) (justify left bottom))
+  )
   (text "James TODO: Verify these are wired correctly" (at 104.14 202.565 0)
     (effects (font (size 1.27 1.27) (color 255 153 0 1)) (justify left bottom))
@@
     (effects (font (size 1.27 1.27)) (justify left bottom))
   )
+  (text "\"The Apple II Circuit Description\" shows multiple \nversions of this part of the schematic.\n\nV0 is much different than V1 and later.\n\n-baldee"
+    (at -48.895 46.355 0)
+    (effects (font (size 1.27 1.27)) (justify left bottom))
+  )
   (text "Flashing timer\nfor flashing chars" (at 194.945 142.24 0)
     (effects (font (size 1.27 1.27)) (justify left bottom))
@@
     (effects (font (size 1.27 1.27)) (justify left bottom))
   )
-  (label "SOFT5-A2-8" (at 370.84 51.435 0) (fields_autoplaced)
-    (effects (font (size 1.27 1.27)) (justify left bottom))
-  )
   (label "14M" (at 384.81 136.525 0) (fields_autoplaced)
     (effects (font (size 1.27 1.27)) (justify left bottom))
@@
     (effects (font (size 1.27 1.27)) (justify right bottom))
   )
-  (label "SOFT5-A2-8" (at 82.55 248.285 180) (fields_autoplaced)
+  (label "SOFT5" (at 82.55 248.285 180) (fields_autoplaced)
     (effects (font (size 1.27 1.27)) (justify right bottom))
   )
-  (label "SOFT5-A2-11" (at 370.84 66.675 0) (fields_autoplaced)
-    (effects (font (size 1.27 1.27)) (justify left bottom))
-  )
   (label "HIRES" (at 186.055 185.42 180) (fields_autoplaced)
     (effects (font (size 1.27 1.27)) (justify right bottom))
@@
     (effects (font (size 1.27 1.27)) (justify left bottom))
   )
+  (label "~{7M}" (at 45.72 163.195 180) (fields_autoplaced)
+    (effects (font (size 1.27 1.27)) (justify right bottom))
+  )
   (label "LD[0..7]" (at 384.175 29.845 0) (fields_autoplaced)
     (effects (font (size 1.27 1.27)) (justify left bottom))
@@
     (effects (font (size 1.27 1.27)) (justify right bottom))
   )
-  (label "SOFT5-A2-11" (at 82.55 263.525 180) (fields_autoplaced)
+  (label "SOFT5" (at 82.55 263.525 180) (fields_autoplaced)
     (effects (font (size 1.27 1.27)) (justify right bottom))
   )
@@
     (effects (font (size 1.27 1.27)) (justify left))
   )
-  (hierarchical_label "SS-Mix_~{NoMix}" (shape input) (at 32.385 191.135 180) (fields_autoplaced)
+  (hierarchical_label "~{7M}" (shape input) (at 32.385 163.195 180) (fields_autoplaced)
     (effects (font (size 1.27 1.27)) (justify right))
   )
-  (hierarchical_label "SOFT5-A2-11" (shape output) (at 387.35 66.675 0) (fields_autoplaced)
-    (effects (font (size 1.27 1.27)) (justify left))
+  (hierarchical_label "SS-Mix_~{NoMix}" (shape input) (at 32.385 191.135 180) (fields_autoplaced)
+    (effects (font (size 1.27 1.27)) (justify right))
   )
   (hierarchical_label "VB" (shape input) (at 22.225 26.035 180) (fields_autoplaced)
@@
     (effects (font (size 1.27 1.27)) (justify right))
   )
-  (hierarchical_label "SOFT5-A2-8" (shape output) (at 387.35 51.435 0) (fields_autoplaced)
-    (effects (font (size 1.27 1.27)) (justify left))
-  )
   (hierarchical_label "H4" (shape input) (at 27.305 74.93 180) (fields_autoplaced)
     (effects (font (size 1.27 1.27)) (justify right))
@@
   (symbol (lib_id "Jumper:SolderJumper_2_Open") (at 62.23 42.545 0) (unit 1)
     (in_bom yes) (on_board yes) (dnp no)
-    (property "Reference" "JP10" (at 62.23 40.259 0)
+    (property "Reference" "JP14" (at 62.23 40.259 0)
       (effects (font (size 1.27 1.27)))
     )
@@
       (project "AppleII+"
         (path "/7f3799a0-e0b6-4ab6-94fe-921c86f8e727/00000000-0000-0000-0000-0000632bf564"
-          (reference "JP10") (unit 1)
+          (reference "JP14") (unit 1)
         )
       )
@@
   (symbol (lib_id "Jumper:SolderJumper_2_Bridged") (at 62.23 50.165 0) (unit 1)
     (in_bom yes) (on_board yes) (dnp no)
-    (property "Reference" "JP11" (at 62.484 48.133 0)
+    (property "Reference" "JP16" (at 62.484 48.133 0)
       (effects (font (size 1.27 1.27)))
     )
@@
       (project "AppleII+"
         (path "/7f3799a0-e0b6-4ab6-94fe-921c86f8e727/00000000-0000-0000-0000-0000632bf564"
-          (reference "JP11") (unit 1)
+          (reference "JP16") (unit 1)
         )
       )
